File: Eagle files/raspi3_nonHatv2.brd (EAGLE design)
At the start: 69.8 x 63.2 mm, 37 parts, among them IC5 PAM8403, K1 PIN20X2

Commit message: 3-Eagle_final
Parts:
- moved THERMISTOR2 48.8 mm to (74.9, 48.3)
- moved THERMISTOR3 48.4 mm to (74.9, 54.0)
- moved POWER 46.1 mm to (74.9, 30.5)
- moved J4 40.9 mm to (6.35, 41.0), turned to 90 degrees
- moved THERMISTOR4 38.9 mm to (73.7, 14.6), turned to 270 degrees
- moved R11 32.5 mm to (42.5, 21.6), turned to 90 degrees
- moved J1 31.8 mm to (74.9, 64.8)
- moved THERMISTOR1 29.6 mm to (74.9, 21.6)
- moved R10 28.0 mm to (42.5, 14.0), turned to 270 degrees
- moved J2 27.6 mm to (74.9, 42.5)
- moved C8 26.7 mm to (44.5, 19.1), turned to 270 degrees
- moved LED1 25.0 mm to (41.9, 63.5), turned to 180 degrees
- moved C7 24.7 mm to (44.5, 15.9), turned to 90 degrees
- moved EN3 19.9 mm to (47.6, 17.8), turned to 270 degrees
- moved C9 19.3 mm to (52.7, 22.2), turned to 180 degrees
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Routing:
- net +5V: track 36.1 -> 177.0 mm, vias 0 -> 4
- net 0CS0: track 0.00 -> 130.2 mm, vias 0 -> 2
- net +3V3: track 101.2 -> 228.5 mm, vias 0 -> 7
- net SDA: track 22.6 -> 110.6 mm, vias 0 -> 2
- net SCL: track 15.8 -> 102.4 mm, vias 0 -> 2
- net 1MISO: track 0.00 -> 74.3 mm, vias 0 -> 2
- net RX: track 8.04 -> 81.4 mm
- net 1CS0: track 0.00 -> 71.0 mm
- net 1MOSI: track 0.00 -> 68.5 mm, vias 0 -> 2
- net GND: track 268.4 -> 334.3 mm
- net TX: track 8.67 -> 74.2 mm
- net 1SCLK: track 0.00 -> 53.4 mm
- net 0SCLK: track 5.08 -> 45.6 mm
- net 0MISO: track 6.13 -> 42.2 mm
- net 0MOSI: track 14.3 -> 49.2 mm
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Other:
- board size 69.8 x 63.2 mm -> 86.3 x 73.3 mm

Commit message: rearranged
Parts:
- moved U$1 55.4 mm to (17.8, 48.3), turned to 270 degrees
- moved J1 5.08 mm to (69.8, 64.8)
- moved J2 5.08 mm to (69.8, 42.5)
- moved POWER 5.08 mm to (69.8, 30.5)
- moved THERMISTOR1 5.08 mm to (69.8, 21.6)
- moved THERMISTOR2 5.08 mm to (69.8, 48.3)
- moved THERMISTOR3 5.08 mm to (69.8, 54.0)
- moved THERMISTOR4 3.81 mm to (69.8, 14.6)
- moved SPEAKER 3.81 mm to (17.1, 5.71)
- moved C7 1.27 mm to (43.2, 15.9)
- moved C8 1.27 mm to (43.2, 19.1)
- moved EN3 1.27 mm to (46.4, 17.8)
- moved OLED_MODULE 1.27 mm to (50.8, 39.4)
- moved R1 1.27 mm to (52.1, 55.9)
- moved R10 1.27 mm to (41.3, 14.0)
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Connections:
- net AIN0: now also J4.1; no longer J4.2
- net AIN1: now also J4.2; no longer J4.1
- net AIN2: now also J4.3; no longer J4.4
- net AIN3: now also J4.4; no longer J4.3
- net CLK: now also K1.7
- net DT: now also K1.15
Routing:
- net 0CS0: track 130.2 -> 118.7 mm
- net SW: track 5.75 -> 17.2 mm
- net DT: track 4.48 -> 15.5 mm
- net +3V3: track 228.5 -> 218.6 mm
- net SDA: track 110.6 -> 101.4 mm
- net SCL: track 102.4 -> 95.7 mm
- net AIN1: track 18.9 -> 12.3 mm
- net CLK: track 4.86 -> 11.2 mm
- net AIN3: track 17.2 -> 11.4 mm
- net 0SCLK: track 45.6 -> 40.2 mm
- net 1MISO: track 74.3 -> 69.3 mm
- net 0MISO: track 42.2 -> 37.1 mm
- net +5V: track 177.0 -> 172.2 mm
- net N$27: track 8.83 -> 13.4 mm
- net 0MOSI: track 49.2 -> 44.9 mm
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Other:
- board size 86.3 x 73.3 mm -> 79.4 x 73.3 mm
