File: Eagle files/raspi3_nonHatv2.brd (EAGLE design)
At the start: 86.3 x 73.3 mm, 37 parts, among them IC5 PAM8403, K1 PIN20X2

Commit message: 4-eagle-final
Parts:
- moved U$1 54.3 mm to (25.4, 30.5), turned to 90 degrees
Routing:
- net 0CS0: track 130.2 -> 128.0 mm
Changed lines of the file:
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@@
 <attribute name="VALUE" x="6.985" y="64.135" size="1.27" layer="27" rot="R180"/>
 </element>
-<element name="U$1" library="namanpuri" package="MAKE-IN-INDIA" value="MAKE-IN-INDIA-LOGO" x="-26.67" y="15.24" smashed="yes"/>
+<element name="U$1" library="namanpuri" package="MAKE-IN-INDIA" value="MAKE-IN-INDIA-LOGO" x="25.4" y="30.48" smashed="yes" rot="R90"/>
 </elements>
 <signals>
@@
 </signal>
 <signal name="N$5">
-<via x="81.915" y="69.85" extent="1-16" drill="2.794" diameter="3.81"/>
+<via x="83.185" y="69.85" extent="1-16" drill="2.794" diameter="3.81"/>
 </signal>
 <signal name="N$6">
-<via x="80.645" y="6.35" extent="1-16" drill="2.794" diameter="3.81"/>
+<via x="83.185" y="3.81" extent="1-16" drill="2.794" diameter="3.81"/>
 </signal>
 <signal name="N$7">
-<via x="3.175" y="6.35" extent="1-16" drill="2.794" diameter="3.81"/>
+<via x="3.175" y="3.81" extent="1-16" drill="2.794" diameter="3.81"/>
 </signal>
 <signal name="0MOSI">
@@
 <contactref element="K1" pad="24"/>
 <contactref element="J2" pad="1"/>
-<wire x1="30.48" y1="36.83" x2="25.4" y2="36.83" width="0.6096" layer="16"/>
-<wire x1="25.4" y1="36.83" x2="24.13" y2="38.1" width="0.6096" layer="16"/>
-<wire x1="24.13" y1="38.1" x2="24.13" y2="65.405" width="0.6096" layer="16"/>
-<wire x1="24.13" y1="65.405" x2="30.0992" y2="71.3742" width="0.6096" layer="16"/>
+<wire x1="24.4475" y1="65.7225" x2="30.0992" y2="71.3742" width="0.6096" layer="16"/>
 <wire x1="30.0992" y1="71.3742" x2="74.93" y2="71.3742" width="0.6096" layer="16"/>
 <wire x1="74.93" y1="42.545" x2="79.375" y2="42.545" width="0.6096" layer="16"/>
@@
 <wire x1="84.6255" y1="42.545" x2="84.3842" y2="42.7863" width="0.6096" layer="16"/>
 <wire x1="84.3842" y1="55.3158" x2="84.3842" y2="42.7863" width="0.6096" layer="16"/>
+<wire x1="30.48" y1="36.83" x2="29.21" y2="36.83" width="0.6096" layer="16"/>
+<wire x1="29.21" y1="36.83" x2="27.94" y2="38.1" width="0.6096" layer="16"/>
+<wire x1="24.13" y1="65.405" x2="24.4475" y2="65.7225" width="0.6096" layer="16"/>
+<wire x1="27.94" y1="38.1" x2="27.94" y2="48.895" width="0.6096" layer="16"/>
+<wire x1="27.94" y1="48.895" x2="24.13" y2="52.705" width="0.6096" layer="16"/>
+<wire x1="24.13" y1="52.705" x2="24.13" y2="65.405" width="0.6096" layer="16"/>
 </signal>
 <signal name="TX">

Commit message: size adjusted
Parts:
- added SL1: (no value), con-amp-quick:05P
- moved J1 6.84 mm to (68.6, 67.3)
- moved THERMISTOR3 6.63 mm to (68.6, 55.9)
- moved THERMISTOR2 6.48 mm to (68.6, 49.5)
- moved J2 6.38 mm to (68.6, 43.2)
- moved POWER 6.35 mm to (68.6, 30.5)
- moved THERMISTOR1 6.35 mm to (68.6, 21.6)
- moved THERMISTOR4 5.08 mm to (68.6, 14.6)
- moved SPEAKER 4.45 mm to (17.1, 5.08)
- moved K1 2.62 mm to (29.2, 32.4)
- moved U$1 2.29 mm to (23.5, 29.2)
- moved C3 1.42 mm to (19.1, 55.2)
- moved C7 0.64 mm to (43.8, 15.9)
- moved C8 0.64 mm to (43.8, 19.1)
- moved R10 0.64 mm to (41.9, 14.0)
- moved R11 0.64 mm to (41.9, 21.6)
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Connections:
- new net 27: K1.27, SL1.2
- new net 29: K1.29, SL1.3
- new net 31: K1.31, SL1.4
- new net 33: K1.33, SL1.5
- net AIN0: now also J4.1; no longer J4.2
- net AIN1: now also J4.2; no longer J4.1
- net AIN2: now also J4.3; no longer J4.4
- net AIN3: now also J4.4; no longer J4.3
- net CLK: now also K1.7
- net DT: now also K1.13
- net GND: now also SL1.1
- net SW: now also K1.15
Routing:
- net SW: track 5.75 -> 30.8 mm, vias 0 -> 2
- net 0CS0: track 128.0 -> 111.8 mm
- net DT: track 4.48 -> 16.9 mm
- net SDA: track 110.6 -> 98.1 mm
- net +5V: track 177.0 -> 166.8 mm
- net GND: track 334.3 -> 344.0 mm
- net CLK: track 4.86 -> 14.1 mm
- net +3V3: track 228.5 -> 219.3 mm, vias 7 -> 6
- net SCL: track 102.4 -> 93.7 mm
- net AIN1: track 18.9 -> 11.7 mm
- net 1CS0: track 71.0 -> 65.5 mm
- net AIN3: track 17.2 -> 11.8 mm
- net N$27: track 8.83 -> 14.0 mm
- net 0SCLK: track 45.6 -> 41.1 mm
- net N$4: track 4.70 -> 9.14 mm
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Other:
- board size 86.3 x 73.3 mm -> 76.2 x 73.3 mm
