File: Eagle files/raspi3_nonHatv2.sch (EAGLE design)
At the start: 37 parts, among them IC5 PAM8403, K1 PIN20X2

Commit message: size adjusted
Parts:
- added SL1: (no value), con-amp-quick:M05
Connections:
- new net 27: K1.27, SL1.2
- new net 29: K1.29, SL1.3
- new net 31: K1.31, SL1.4
- new net 33: K1.33, SL1.5
- net AIN0: now also J4.1; no longer J4.2
- net AIN1: now also J4.2; no longer J4.1
- net AIN2: now also J4.3; no longer J4.4
- net AIN3: now also J4.4; no longer J4.3
- net CLK: now also K1.7
- net DT: now also K1.13
- net GND: now also SL1.1
- net SW: now also K1.15
Other:
- note added: "Notes: 1. Check package of JSTs 3. Check quatity of 4 pin jst"
- note removed: "Notes: 1. Check package of JSTs 2. Do connections of Rotary Encoder 3. Check quatity of 4 pin jst"
- moved on the sheet: J4
Changed lines of the file:
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@@
 <?xml version="1.0" encoding="utf-8"?>
 <!DOCTYPE eagle SYSTEM "eagle.dtd">
-<eagle version="9.6.2">
+<eagle version="9.4.1">
 <drawing>
 <settings>
@@
 <part name="+3V11" library="supply1" deviceset="+3V3" device=""/>
 <part name="U$1" library="namanpuri" deviceset="MAKE-IN-INDIA-LOGO" device=""/>
+<part name="SL1" library="con-amp-quick" library_urn="urn:adsk.eagle:library:125" deviceset="M05" device="" package3d_urn="urn:adsk.eagle:package:5961/1"/>
+<part name="GND8" library="MSP PROJECT LIBRARY" deviceset="GND" device=""/>
 </parts>
 <sheets>
@@
 <text x="-92.71" y="118.11" size="1.778" layer="91">Notes:
 1. Check package of JSTs
-2. Do connections of Rotary Encoder
 3. Check quatity of 4 pin jst</text>
 <text x="-25.4" y="130.81" size="2.54" layer="91" font="vector" ratio="17">ROTARY ENCODER</text>
@@
 <attribute name="NAME" x="-19.05" y="5.588" size="1.778" layer="95" font="vector"/>
 </instance>
-<instance part="J4" gate="G$1" x="133.35" y="44.45" smashed="yes">
-<attribute name="VALUE" x="128.27" y="37.084" size="1.778" layer="96" font="vector"/>
-<attribute name="NAME" x="128.27" y="52.578" size="1.778" layer="95" font="vector"/>
+<instance part="J4" gate="G$1" x="13.97" y="-2.54" smashed="yes">
+<attribute name="VALUE" x="8.89" y="-9.906" size="1.778" layer="96" font="vector"/>
+<attribute name="NAME" x="8.89" y="5.588" size="1.778" layer="95" font="vector"/>
 </instance>
 <instance part="U$3" gate="G$1" x="111.76" y="49.53" smashed="yes">
@@
 </instance>
 <instance part="U$1" gate="G$1" x="113.03" y="121.92" smashed="yes"/>
+<instance part="SL1" gate="G$1" x="34.29" y="0" smashed="yes">
+<attribute name="VALUE" x="31.75" y="-10.16" size="1.778" layer="96"/>
+<attribute name="NAME" x="31.75" y="8.382" size="1.778" layer="95"/>
+</instance>
+<instance part="GND8" gate="1" x="43.18" y="-8.89" smashed="yes">
+<attribute name="VALUE" x="40.64" y="-11.43" size="1.778" layer="96"/>
+</instance>
 </instances>
 <busses>
@@
 <wire x1="82.55" y1="60.96" x2="74.93" y2="60.96" width="0.1524" layer="91"/>
 <junction x="74.93" y="60.96"/>
+</segment>
+<segment>
+<pinref part="SL1" gate="G$1" pin="1"/>
+<wire x1="41.91" y1="-5.08" x2="43.18" y2="-5.08" width="0.1524" layer="91"/>
+<pinref part="GND8" gate="1" pin="GND"/>
+<wire x1="43.18" y1="-5.08" x2="43.18" y2="-6.35" width="0.1524" layer="91"/>
 </segment>
 </net>
@@
 <label x="-34.29" y="119.38" size="1.27" layer="95" font="vector" ratio="17" rot="R90" xref="yes"/>
 </segment>
+<segment>
+<wire x1="36.83" y1="55.88" x2="35.56" y2="55.88" width="0.1524" layer="91" style="dashdot"/>
+<wire x1="35.56" y1="55.88" x2="30.48" y2="55.88" width="0.1524" layer="91" curve="180"/>
+<wire x1="30.48" y1="55.88" x2="29.21" y2="55.88" width="0.1524" layer="91"/>
+<pinref part="K1" gate="G$1" pin="13"/>
+<label x="27.94" y="55.88" size="1.27" layer="95" font="vector" ratio="16" rot="R180" xref="yes"/>
+</segment>
 </net>
 <net name="CLK" class="0">
@@
 <label x="-41.91" y="119.38" size="1.27" layer="95" font="vector" ratio="17" rot="R90" xref="yes"/>
 </segment>
+<segment>
+<wire x1="36.83" y1="63.5" x2="33.02" y2="63.5" width="0.1524" layer="91"/>
+<wire x1="33.02" y1="63.5" x2="30.48" y2="63.5" width="0.1524" layer="91" curve="180"/>
+<wire x1="30.48" y1="63.5" x2="29.21" y2="63.5" width="0.1524" layer="91"/>
+<pinref part="K1" gate="G$1" pin="7"/>
+<label x="27.94" y="63.5" size="1.27" layer="95" font="vector" ratio="16" rot="R180" xref="yes"/>
+</segment>
 </net>
 <net name="SW" class="0">
@@
 <wire x1="-26.67" y1="118.11" x2="-26.67" y2="115.57" width="0.1524" layer="91"/>
 <label x="-26.67" y="119.38" size="1.27" layer="95" font="vector" ratio="17" rot="R90" xref="yes"/>
+</segment>
+<segment>
+<wire x1="36.83" y1="53.34" x2="35.56" y2="53.34" width="0.1524" layer="91" style="dashdot"/>
+<pinref part="K1" gate="G$1" pin="15"/>
+<wire x1="35.56" y1="53.34" x2="30.48" y2="53.34" width="0.1524" layer="91" curve="180"/>
+<wire x1="30.48" y1="53.34" x2="29.21" y2="53.34" width="0.1524" layer="91"/>
+<label x="27.94" y="53.34" size="1.27" layer="95" font="vector" ratio="16" rot="R180" xref="yes"/>
 </segment>
 </net>
@@
 </segment>
 <segment>
-<pinref part="J4" gate="G$1" pin="2"/>
-<wire x1="138.43" y1="44.45" x2="139.7" y2="44.45" width="0.1524" layer="91"/>
-<label x="140.97" y="44.45" size="1.27" layer="95" font="vector" ratio="16" xref="yes"/>
+<pinref part="J4" gate="G$1" pin="1"/>
+<wire x1="19.05" y1="-5.08" x2="20.32" y2="-5.08" width="0.1524" layer="91"/>
+<label x="21.59" y="-5.08" size="1.27" layer="95" font="vector" ratio="16" xref="yes"/>
 </segment>
 </net>
@@
 </segment>
 <segment>
-<pinref part="J4" gate="G$1" pin="1"/>
-<wire x1="138.43" y1="41.91" x2="139.7" y2="41.91" width="0.1524" layer="91"/>
-<label x="140.97" y="41.91" size="1.27" layer="95" font="vector" ratio="16" xref="yes"/>
+<pinref part="J4" gate="G$1" pin="2"/>
+<wire x1="19.05" y1="-2.54" x2="20.32" y2="-2.54" width="0.1524" layer="91"/>
+<label x="21.59" y="-2.54" size="1.27" layer="95" font="vector" ratio="16" xref="yes"/>
 </segment>
 </net>
@@
 </segment>
 <segment>
-<pinref part="J4" gate="G$1" pin="4"/>
-<wire x1="138.43" y1="49.53" x2="139.7" y2="49.53" width="0.1524" layer="91"/>
-<label x="140.97" y="49.53" size="1.27" layer="95" font="vector" ratio="16" xref="yes"/>
+<pinref part="J4" gate="G$1" pin="3"/>
+<wire x1="19.05" y1="0" x2="20.32" y2="0" width="0.1524" layer="91"/>
+<label x="21.59" y="0" size="1.27" layer="95" font="vector" ratio="16" xref="yes"/>
 </segment>
 </net>
@@
 </segment>
 <segment>
-<pinref part="J4" gate="G$1" pin="3"/>
-<wire x1="138.43" y1="46.99" x2="139.7" y2="46.99" width="0.1524" layer="91"/>
-<label x="140.97" y="46.99" size="1.27" layer="95" font="vector" ratio="16" xref="yes"/>
+<pinref part="J4" gate="G$1" pin="4"/>
+<wire x1="19.05" y1="2.54" x2="20.32" y2="2.54" width="0.1524" layer="91"/>
+<label x="21.59" y="2.54" size="1.27" layer="95" font="vector" ratio="16" xref="yes"/>
 </segment>
 </net>
@@
 </segment>
 </net>
+<net name="27" class="0">
+<segment>
+<pinref part="SL1" gate="G$1" pin="2"/>
+<wire x1="41.91" y1="-2.54" x2="43.18" y2="-2.54" width="0.1524" layer="91"/>
+<label x="44.45" y="-2.54" size="1.27" layer="95" font="vector" ratio="16" xref="yes"/>
+</segment>
+<segment>
+<wire x1="36.83" y1="38.1" x2="35.56" y2="38.1" width="0.1524" layer="91" style="dashdot"/>
+<wire x1="35.56" y1="38.1" x2="33.02" y2="38.1" width="0.1524" layer="91" curve="180"/>
+<wire x1="33.02" y1="38.1" x2="31.75" y2="38.1" width="0.1524" layer="91" style="dashdot"/>
+<pinref part="K1" gate="G$1" pin="27"/>
+<label x="30.48" y="38.1" size="1.27" layer="95" font="vector" ratio="16" rot="R180" xref="yes"/>
+</segment>
+</net>
+<net name="29" class="0">
+<segment>
+<pinref part="SL1" gate="G$1" pin="3"/>
+<wire x1="41.91" y1="0" x2="43.18" y2="0" width="0.1524" layer="91"/>
+<label x="44.45" y="0" size="1.27" layer="95" font="vector" ratio="16" xref="yes"/>
+</segment>
+<segment>
+<wire x1="36.83" y1="35.56" x2="35.56" y2="35.56" width="0.1524" layer="91" style="dashdot"/>
+<wire x1="35.56" y1="35.56" x2="33.02" y2="35.56" width="0.1524" layer="91" curve="180"/>
+<wire x1="33.02" y1="35.56" x2="31.75" y2="35.56" width="0.1524" layer="91" style="dashdot"/>
+<pinref part="K1" gate="G$1" pin="29"/>
+<label x="30.48" y="35.56" size="1.27" layer="95" font="vector" ratio="16" rot="R180" xref="yes"/>
+</segment>
+</net>
+<net name="31" class="0">
+<segment>
+<pinref part="SL1" gate="G$1" pin="4"/>
+<wire x1="41.91" y1="2.54" x2="43.18" y2="2.54" width="0.1524" layer="91"/>
+<label x="44.45" y="2.54" size="1.27" layer="95" font="vector" ratio="16" xref="yes"/>
+</segment>
+<segment>
+<wire x1="36.83" y1="33.02" x2="35.56" y2="33.02" width="0.1524" layer="91" style="dashdot"/>
+<wire x1="35.56" y1="33.02" x2="33.02" y2="33.02" width="0.1524" layer="91" curve="180"/>
+<wire x1="33.02" y1="33.02" x2="31.75" y2="33.02" width="0.1524" layer="91" style="dashdot"/>
+<pinref part="K1" gate="G$1" pin="31"/>
+<label x="30.48" y="33.02" size="1.27" layer="95" font="vector" ratio="16" rot="R180" xref="yes"/>
+</segment>
+</net>
+<net name="33" class="0">
+<segment>
+<pinref part="SL1" gate="G$1" pin="5"/>
+<wire x1="41.91" y1="5.08" x2="43.18" y2="5.08" width="0.1524" layer="91"/>
+<label x="44.45" y="5.08" size="1.27" layer="95" font="vector" ratio="16" xref="yes"/>
+</segment>
+<segment>
+<wire x1="36.83" y1="30.48" x2="35.56" y2="30.48" width="0.1524" layer="91" style="dashdot"/>
+<wire x1="35.56" y1="30.48" x2="33.02" y2="30.48" width="0.1524" layer="91" curve="180"/>
+<wire x1="33.02" y1="30.48" x2="31.75" y2="30.48" width="0.1524" layer="91" style="dashdot"/>
+<pinref part="K1" gate="G$1" pin="33"/>
+<label x="30.48" y="30.48" size="1.27" layer="95" font="vector" ratio="16" rot="R180" xref="yes"/>
+</segment>
+</net>
