File: Eagle files/raspi3_nonHatv2.sch (EAGLE design)
At the start: 40 parts, among them IC5 PAM8403, K1 PIN20X2, X1 JST-XH-05-PIN-LONG-PAD, X2 JST-XH-02-PIN-LONG-PAD

Commit message: updated
Parts:
- removed J4: (no value), SparkFun-Connectors:CONN_04POLAR
- removed THERMISTOR1, THERMISTOR2, THERMISTOR3, THERMISTOR4: (no value), SparkFun-Connectors:CONN_02POLAR
- added X3, X4, X5: JST-XH-02-PIN-LONG-PAD, Rembrandt Electronics - JST XH Connectors v1-0:JST-XH-02-PIN-LONG-PAD
Connections:
- net +3V3: now also X4-1.S; no longer THERMISTOR2.1
- net +5V: now also X5-1.S; no longer THERMISTOR3.1
- net AIN0: now also X1-4.S; no longer J4.1
- net AIN1: now also X1-3.S; no longer J4.2
- net AIN2: now also X1-2.S; no longer J4.3
- net AIN3: now also X1-1.S; no longer J4.4
- net GND: now also X1-5.S, X4-2.S, X5-2.S; no longer THERMISTOR2.2, THERMISTOR3.2
- net RX: now also X3-2.S; no longer THERMISTOR4.2
- net SCL: now also X2-1.S; no longer THERMISTOR1.1
- net SDA: now also X2-2.S; no longer THERMISTOR1.2
- net TX: now also X3-1.S; no longer THERMISTOR4.1
Other:
- moved on the sheet: X2-1, X2-2

Commit message: 8-eagle
Parts:
- removed J1, J2: (no value), SparkFun-Connectors:CONN_04POLAR
- added X6, X7: JST-XH-03-PIN-LONG-PAD, Rembrandt Electronics - JST XH Connectors v1-0:JST-XH-03-PIN-LONG-PAD
- added X8, X9: JST-XH-05-PIN-LONG-PAD, Rembrandt Electronics - JST XH Connectors v1-0:JST-XH-05-PIN-LONG-PAD
Connections:
- new net GND1: X8-5.S
- new net GND2: X9-5.S
- new net N$10: X6-3.S
- new net N$8: X6-1.S
- new net N$9: X6-2.S
- net 0CS0: now also X8-4.S; no longer J2.1
- net 0MISO: now also X8-1.S; no longer J2.4
- net 0MOSI: now also X8-2.S; no longer J2.3
- net 0SCLK: now also X8-3.S; no longer J2.2
- net 1CS0: now also X9-4.S; no longer J1.1
- net 1MISO: now also X9-1.S; no longer J1.4
- net 1MOSI: now also X9-2.S; no longer J1.3
- net 1SCLK: now also X9-3.S; no longer J1.2

Commit message: raspi material added
Parts:
- removed POWER: (no value), SparkFun-Connectors:CONN_03POLAR
- removed X6: JST-XH-03-PIN-LONG-PAD, Rembrandt Electronics - JST XH Connectors v1-0:JST-XH-03-PIN-LONG-PAD
Connections:
- removed net GND1: X8-5.S
- removed net GND2: X9-5.S
- removed net N$10: X6-3.S
- removed net N$8: X6-1.S
- removed net N$9: X6-2.S
- net +3V3: now also X7-2.S; no longer POWER.2
- net +5V: now also X7-3.S; no longer POWER.3
- net GND: now also X7-1.S, X8-5.S, X9-5.S; no longer POWER.1
Changed lines of the file:
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@@
 <?xml version="1.0" encoding="utf-8"?>
 <!DOCTYPE eagle SYSTEM "eagle.dtd">
-<eagle version="9.6.2">
+<eagle version="9.4.1">
 <drawing>
 <settings>
@@
 <part name="P+7" library="supply1" deviceset="+5V" device=""/>
 <part name="GND5" library="MSP PROJECT LIBRARY" deviceset="GND" device=""/>
-<part name="POWER" library="SparkFun-Connectors" library_urn="urn:adsk.eagle:library:513" deviceset="CONN_03" device="POLAR" package3d_urn="urn:adsk.eagle:package:38064/1"/>
-<part name="P+4" library="supply1" deviceset="+5V" device=""/>
-<part name="GND6" library="MSP PROJECT LIBRARY" deviceset="GND" device=""/>
-<part name="+3V4" library="supply1" deviceset="+3V3" device=""/>
 <part name="EN3" library="Encoders" library_urn="urn:adsk.eagle:library:14555662" deviceset="PEC11L-4220F-S0015" device="" package3d_urn="urn:adsk.eagle:package:14522106/4"/>
 <part name="C7" library="adafruit" deviceset="C-US" device="C0603K"/>
@@
 <part name="GND7" library="MSP PROJECT LIBRARY" deviceset="GND" device=""/>
 <part name="P+2" library="supply1" deviceset="+5V" device=""/>
-<part name="X6" library="Rembrandt Electronics - JST XH Connectors v1-0" deviceset="JST-XH-03-PIN" device="-LONG-PAD"/>
 <part name="X7" library="Rembrandt Electronics - JST XH Connectors v1-0" deviceset="JST-XH-03-PIN" device="-LONG-PAD"/>
 <part name="X8" library="Rembrandt Electronics - JST XH Connectors v1-0" deviceset="JST-XH-05-PIN" device="-LONG-PAD"/>
 <part name="X9" library="Rembrandt Electronics - JST XH Connectors v1-0" deviceset="JST-XH-05-PIN" device="-LONG-PAD"/>
+<part name="GND13" library="SparkFun-PowerSymbols" library_urn="urn:adsk.eagle:library:530" deviceset="GND" device=""/>
+<part name="+3V5" library="supply1" deviceset="+3V3" device=""/>
+<part name="P+6" library="supply1" deviceset="+5V" device=""/>
+<part name="GND6" library="MSP PROJECT LIBRARY" deviceset="GND" device=""/>
+<part name="GND14" library="MSP PROJECT LIBRARY" deviceset="GND" device=""/>
 </parts>
 <sheets>
@@
 <attribute name="VALUE" x="-41.91" y="38.1" size="1.778" layer="96"/>
 </instance>
-<instance part="POWER" gate="J$1" x="-36.83" y="16.51" smashed="yes">
-<attribute name="VALUE" x="-39.37" y="9.144" size="1.778" layer="96" font="vector"/>
-</instance>
-<instance part="P+4" gate="1" x="-27.94" y="22.86" smashed="yes">
-<attribute name="VALUE" x="-26.67" y="25.4" size="1.778" layer="96" rot="R180"/>
-</instance>
-<instance part="GND6" gate="1" x="-27.94" y="10.16" smashed="yes">
-<attribute name="VALUE" x="-30.48" y="7.62" size="1.778" layer="96"/>
-</instance>
-<instance part="+3V4" gate="G$1" x="-22.86" y="20.32" smashed="yes">
-<attribute name="VALUE" x="-20.32" y="22.86" size="1.778" layer="96" rot="R180"/>
-</instance>
 <instance part="EN3" gate="G$1" x="3.81" y="104.14" smashed="yes">
 <attribute name="NAME" x="-1.27" y="112.268" size="1.778" layer="95"/>
@@
 <attribute name="VALUE" x="-22.86" y="-6.35" size="1.778" layer="96" rot="R180"/>
 </instance>
-<instance part="X6" gate="-1" x="101.6" y="2.54" smashed="yes">
-<attribute name="NAME" x="104.14" y="1.778" size="1.524" layer="95"/>
-<attribute name="VALUE" x="100.838" y="3.937" size="1.778" layer="96"/>
-</instance>
-<instance part="X6" gate="-2" x="101.6" y="0" smashed="yes">
-<attribute name="NAME" x="104.14" y="-0.762" size="1.524" layer="95"/>
-</instance>
-<instance part="X6" gate="-3" x="101.6" y="-2.54" smashed="yes">
-<attribute name="NAME" x="104.14" y="-3.302" size="1.524" layer="95"/>
-</instance>
 <instance part="X7" gate="-1" x="129.54" y="15.24" smashed="yes">
 <attribute name="NAME" x="132.08" y="14.478" size="1.524" layer="95"/>
@@
 <instance part="X9" gate="-5" x="48.26" y="-35.56" smashed="yes">
 <attribute name="NAME" x="50.8" y="-36.322" size="1.524" layer="95"/>
+</instance>
+<instance part="GND13" gate="1" x="124.46" y="20.32" smashed="yes">
+<attribute name="VALUE" x="124.46" y="20.066" size="1.778" layer="96" align="top-center"/>
+</instance>
+<instance part="+3V5" gate="G$1" x="123.19" y="16.51" smashed="yes">
+<attribute name="VALUE" x="120.65" y="16.51" size="1.778" layer="96" rot="R180"/>
+</instance>
+<instance part="P+6" gate="1" x="119.38" y="13.97" smashed="yes">
+<attribute name="VALUE" x="116.84" y="15.24" size="1.778" layer="96" rot="R180"/>
+</instance>
+<instance part="GND6" gate="1" x="43.18" y="-39.37" smashed="yes">
+<attribute name="VALUE" x="40.64" y="-41.91" size="1.778" layer="96"/>
+</instance>
+<instance part="GND14" gate="1" x="69.85" y="-38.1" smashed="yes">
+<attribute name="VALUE" x="67.31" y="-40.64" size="1.778" layer="96"/>
 </instance>
 </instances>
@@
 </segment>
 <segment>
-<wire x1="-29.21" y1="13.97" x2="-27.94" y2="13.97" width="0.1524" layer="91"/>
-<pinref part="POWER" gate="J$1" pin="1"/>
-<pinref part="GND6" gate="1" pin="GND"/>
-<wire x1="-27.94" y1="13.97" x2="-27.94" y2="12.7" width="0.1524" layer="91"/>
-</segment>
-<segment>
 <pinref part="A1" gate="G$1" pin="SLEEVE"/>
 <wire x1="3.81" y1="39.37" x2="2.54" y2="39.37" width="0.1524" layer="91" style="dashdot"/>
@@
 <label x="58.42" y="-6.35" size="1.27" layer="95" font="vector" ratio="16" rot="R180" xref="yes"/>
 </segment>
+<segment>
+<pinref part="GND13" gate="1" pin="GND"/>
+<pinref part="X7" gate="-1" pin="S"/>
+<wire x1="124.46" y1="22.86" x2="127" y2="22.86" width="0.1524" layer="91"/>
+<wire x1="127" y1="22.86" x2="127" y2="15.24" width="0.1524" layer="91"/>
+</segment>
+<segment>
+<pinref part="GND6" gate="1" pin="GND"/>
+<wire x1="43.18" y1="-36.83" x2="43.18" y2="-35.56" width="0.1524" layer="91"/>
+<pinref part="X9" gate="-5" pin="S"/>
+<wire x1="45.72" y1="-35.56" x2="44.45" y2="-35.56" width="0.1524" layer="91"/>
+<wire x1="43.18" y1="-35.56" x2="45.72" y2="-35.56" width="0.1524" layer="91"/>
+<junction x="45.72" y="-35.56"/>
+</segment>
+<segment>
+<pinref part="X8" gate="-5" pin="S"/>
+<wire x1="71.12" y1="-35.56" x2="69.85" y2="-35.56" width="0.1524" layer="91"/>
+<pinref part="GND14" gate="1" pin="GND"/>
+</segment>
 </net>
 <net name="+3V3" class="0">
@@
 <junction x="90.17" y="118.11"/>
 <wire x1="90.17" y1="121.92" x2="90.17" y2="118.11" width="0.1524" layer="91"/>
-</segment>
-<segment>
-<pinref part="POWER" gate="J$1" pin="2"/>
-<pinref part="+3V4" gate="G$1" pin="+3V3"/>
-<wire x1="-22.86" y1="17.78" x2="-22.86" y2="16.51" width="0.1524" layer="91"/>
-<wire x1="-22.86" y1="16.51" x2="-29.21" y2="16.51" width="0.1524" layer="91"/>
 </segment>
 <segment>
@@
 <pinref part="+3V12" gate="G$1" pin="+3V3"/>
 <wire x1="81.28" y1="-11.43" x2="81.28" y2="-12.7" width="0.1524" layer="91"/>
+</segment>
+<segment>
+<pinref part="+3V5" gate="G$1" pin="+3V3"/>
+<pinref part="X7" gate="-2" pin="S"/>
+<wire x1="123.19" y1="13.97" x2="123.19" y2="12.7" width="0.1524" layer="91"/>
+<wire x1="123.19" y1="12.7" x2="127" y2="12.7" width="0.1524" layer="91"/>
 </segment>
 </net>
@@
 </segment>
 <segment>
-<wire x1="-27.94" y1="19.05" x2="-29.21" y2="19.05" width="0.1524" layer="91"/>
-<pinref part="POWER" gate="J$1" pin="3"/>
-<pinref part="P+4" gate="1" pin="+5V"/>
-<wire x1="-27.94" y1="20.32" x2="-27.94" y2="19.05" width="0.1524" layer="91"/>
-</segment>
-<segment>
 <pinref part="X5" gate="-1" pin="S"/>
 <wire x1="-24.13" y1="-12.7" x2="-25.4" y2="-12.7" width="0.1524" layer="91"/>
 <wire x1="-25.4" y1="-11.43" x2="-25.4" y2="-12.7" width="0.1524" layer="91"/>
 <pinref part="P+2" gate="1" pin="+5V"/>
+</segment>
+<segment>
+<pinref part="P+6" gate="1" pin="+5V"/>
+<wire x1="119.38" y1="11.43" x2="119.38" y2="10.16" width="0.1524" layer="91"/>
+<pinref part="X7" gate="-3" pin="S"/>
+<wire x1="119.38" y1="10.16" x2="127" y2="10.16" width="0.1524" layer="91"/>
 </segment>
 </net>
@@
 <pinref part="X9" gate="-3" pin="S"/>
 <wire x1="45.72" y1="-30.48" x2="44.45" y2="-30.48" width="0.1524" layer="91"/>
-<label x="40.64" y="-30.48" size="1.27" layer="95" font="vector" ratio="16" rot="R180" xref="yes"/>
+<label x="41.91" y="-30.48" size="1.27" layer="95" font="vector" ratio="16" rot="R180" xref="yes"/>
 </segment>
 </net>
@@
 <pinref part="X9" gate="-4" pin="S"/>
 <wire x1="45.72" y1="-33.02" x2="44.45" y2="-33.02" width="0.1524" layer="91"/>
-<label x="40.64" y="-33.02" size="1.27" layer="95" font="vector" ratio="16" rot="R180" xref="yes"/>
+<label x="41.91" y="-33.02" size="1.27" layer="95" font="vector" ratio="16" rot="R180" xref="yes"/>
 </segment>
 </net>
@@
 </segment>
 </net>
-<net name="N$8" class="0">
-<segment>
-<pinref part="X6" gate="-1" pin="S"/>
-<wire x1="99.06" y1="2.54" x2="97.79" y2="2.54" width="0.1524" layer="91"/>
-<label x="95.25" y="2.54" size="1.27" layer="95" font="vector" ratio="16" rot="R180" xref="yes"/>
-</segment>
-</net>
-<net name="N$9" class="0">
-<segment>
-<pinref part="X6" gate="-2" pin="S"/>
-<wire x1="99.06" y1="0" x2="97.79" y2="0" width="0.1524" layer="91"/>
-<label x="95.25" y="0" size="1.27" layer="95" font="vector" ratio="16" rot="R180" xref="yes"/>
-</segment>
-</net>
-<net name="N$10" class="0">
-<segment>
-<pinref part="X6" gate="-3" pin="S"/>
-<wire x1="99.06" y1="-2.54" x2="97.79" y2="-2.54" width="0.1524" layer="91"/>
-<label x="96.52" y="-2.54" size="1.27" layer="95" font="vector" ratio="16" rot="R180" xref="yes"/>
-</segment>
-</net>
-<net name="GND1" class="0">
-<segment>
-<pinref part="X8" gate="-5" pin="S"/>
-<wire x1="71.12" y1="-35.56" x2="69.85" y2="-35.56" width="0.1524" layer="91"/>
-<label x="68.58" y="-35.56" size="1.27" layer="95" font="vector" ratio="16" rot="R180" xref="yes"/>
-</segment>
-</net>
-<net name="GND2" class="0">
-<segment>
-<pinref part="X9" gate="-5" pin="S"/>
-<wire x1="45.72" y1="-35.56" x2="44.45" y2="-35.56" width="0.1524" layer="91"/>
-<label x="40.64" y="-35.56" size="1.27" layer="95" font="vector" ratio="16" rot="R180" xref="yes"/>
-</segment>
-</net>
